File: AITLabSmartPursePCB/PurseBoard.sch (KiCad schematic (older format))
At the start: 18 parts, among them IC1 ATMega328PU, IC2 TCA9546A

Commit message: Added pcb schematic updates and attempted FPGA code
This contains the code written this week as well as the hardware design for the smartpurse pcb board
Parts:
- removed PogoPinISR: Conn_01x06, symbol Connector_Generic:Conn_01x06
- added 3.5VBuckC1, 328pC1, 328pC2, Ferrite1C1, Limiter1C2, Limiter2C1, Limiter2C2, LuxAC1, LuxBC1, LuxCC1, LuxDC1, RotEncC1, TempAC1, TempBC1, TempCC1, TempDC1: 0.1uF, symbol Device:C_Small
- added 3.5VBuckC2, 3.5VBuckC3, 3.5VBuckC4, Ferrite1C2: 10uF, symbol Device:C_Small
- added 3.5VBuckL1: 4.7uH 18mOhm, symbol Device:L_Small
- added 3.5VBuckR1, ProgrammerR1: 10kOhm, symbol Device:R_Small
- added 3.5VBuckR1: 20kOhm, symbol Device:R_Small
- added 3.5VBuckR2: 36.5kOhm, symbol Device:R_Small
- added 3VLDOC1, 3VLDOC2, EnumC1, EnumC2, EnumC3, HallC1, Limiter1C1, ProgrammerC2 (x2): 1uF, symbol Device:C_Small
- added D? (x2): LED, symbol Device:LED
- added EnumC4, EnumC5: 22pF, symbol Device:C_Small
- added EnumCrystal1: 16MHz, symbol Device:Crystal_GND24
- added EnumR1, Limiter1R1, Limiter1R3, Limiter1R?, Limiter2R1: 10kΩ, symbol Device:R_Small
- added EnumR2, EnumR3, EnumR? (x2): 22Ω, symbol Device:R_Small
- added FB1: 115 Ohms at 100MHz, symbol Device:Ferrite_Bead_Small
- added HE1: HeatingElement, symbol Device:Heater
- added HeaterR1, HeaterR3: 100Ω, symbol Device:R_Small
- added HeaterR2, HeaterR4: 1MΩ, symbol Device:R_Small
- added IC10: TPS561208DDCR_BuckConverter, symbol MyPartsLibrary:TPS561208DDCR_BuckConverter
- added IC11: TLV1117LV30DCYR_3V_LDO, symbol MyPartsLibrary:TLV1117LV30DCYR_3V_LDO
- added IC12, IC14, IC16, IC18: TC74_TempSensor, symbol MyPartsLibrary:TC74_TempSensor
- added IC13, IC15, IC17, IC19: VEML7700, symbol MyPartsLibrary:VEML7700
- added IC3: AON7810MOSFET, symbol MyPartsLibrary:AON7810MOSFET
- added IC4, IC6: NCP380CurrentLimiter, symbol MyPartsLibrary:NCP380CurrentLimiter
- added IC5, IC7: BSS84-7-F_PChannelMOSFET, symbol MyPartsLibrary:BSS84-7-F_PChannelMOSFET
- added IC8: NSP4201MR6T1G_TVSDiode, symbol MyPartsLibrary:NSP4201MR6T1G_TVSDiode
- added IC9: ATMega16U2_TQFP32, symbol MyPartsLibrary:ATMega16U2_TQFP32
- added J?: USB_A, symbol Connector:USB_A
- added J? (x3), PogoPinISR3: Conn_01x06, symbol Connector_Generic:Conn_01x06
- added J? (x2): Conn_01x04, symbol Connector_Generic:Conn_01x04
- added Limiter1C3: 0.01uF, symbol Device:C_Small
- added Limiter1R4, Limiter2R4: 140Ω, symbol Device:R_Small
- added LuxSensorA2, LuxSensorB1, LuxSensorB2, LuxSensorC1, LuxSensorC2, LuxSensorD1, LuxSensorD2, TempSensorA2, TempSensorB1 (x2), TempSensorC1, TempSensorC2, TempSensorD1, TempSensorD2: Conn_01x05, symbol Connector_Generic:Conn_01x05
- added PogoPinISR1, PogoPinISR2: Conn_01x07, symbol Connector_Generic:Conn_01x07
- added R? (x5), RotEncR5, RotEncR6, RotEncR? (x7): R_Small, symbol Device:R_Small
- added R? (x2): Limiter1R2, symbol Device:R_Small
- added RotEncC4, RotEncC? (x2): C_Small, symbol Device:C_Small
- added SW1, SW2, SW?: SW_SPST, symbol Switch:SW_SPST
- added SW3, SW4: SW_Push, symbol Switch:SW_Push
- added SW5: PEC11L-4215F-S0015 Rotary Encoder Switch, symbol Device:Rotary_Encoder_Switch
- added U?: SN74LVC3G14DCUR_InvertingSchmittTrigger, symbol MyPartsLibrary:SN74LVC3G14DCUR_InvertingSchmittTrigger
- added U?: DRV5032_HallEffectSensor, symbol MyPartsLibrary:DRV5032_HallEffectSensor
- added U?: TXB0104PWR_LevelShifter, symbol MyPartsLibrary:TXB0104PWR_LevelShifter
- added USBR1: 10Ω, symbol Device:R_Small
- I2CHubR1, I2CHubR2: value 10kOhm -> 10kΩ
- renumbered LuxSensor0 to LuxSensorA1, TempSensor0 to TempSensorA1
Connections:
- net 3V: now also IC1.20 (AVCC), IC1.21 (AREF), IC1.7 (VCC), LuxSensorA1.3 (Pin_3), TempSensorA1.3 (Pin_3), 328pC1.1, 328pC2.1, 3VLDOC2.1, IC11.2 (Output), IC11.4 (Output), J?.2 (Pin_2), J?.4 (Pin_4), LuxSensorB1.3 (Pin_3), LuxSensorC1.3 (Pin_3), LuxSensorD1.3 (Pin_3), PogoPinISR1.7 (Pin_7), R?.1, R?.1, R?.1, R?.1, R?.1, RotEncC1.1, RotEncR6.1, RotEncR?.1, RotEncR?.1, TempSensorB1.3 (Pin_3), TempSensorC1.3 (Pin_3), TempSensorD1.3 (Pin_3), U?.8 (Vcc)
- net GNDREF: now also IC1.22 (GND), IC1.8 (GND), LuxSensorA1.4 (Pin_4), LuxSensorA1.5 (Pin_5), TempSensorA1.4 (Pin_4), TempSensorA1.5 (Pin_5), 3.5VBuckC2.2, 3.5VBuckC3.2, 3.5VBuckC4.2, 3.5VBuckR1.2, 328pC1.2, 328pC2.2, 3VLDOC1.2, 3VLDOC2.2, EnumC1.2, EnumC2.2, EnumC3.2, EnumC4.2, EnumC5.2, EnumCrystal1.2, EnumCrystal1.4, Ferrite1C1.2, Ferrite1C2.2, HeaterR2.2, HeaterR4.1, IC10.1 (GND), IC11.1 (GND), IC3.5 (D2), IC3.6 (D2), IC4.5 (GND), IC6.5 (GND), IC8.2 (Vn(GND)), IC9.28 (UGND), IC9.3 (GND), J?.3 (Pin_3), J?.4 (GND), J?.4 (Pin_4), J?.5 (Pin_5), J?.6 (Pin_6), Limiter1C1.2, Limiter1C2.2, Limiter1C3.2, Limiter1R3.2, Limiter1R4.2, Limiter1R?.2, Limiter2C1.2, Limiter2C2.2, Limiter2R4.2, LuxSensorB1.4 (Pin_4), LuxSensorB1.5 (Pin_5), LuxSensorC1.4 (Pin_4), LuxSensorC1.5 (Pin_5), LuxSensorD1.4 (Pin_4), LuxSensorD1.5 (Pin_5), PogoPinISR1.6 (Pin_6), PogoPinISR3.6 (Pin_6), R?.2, R?.2, RotEncC1.2, RotEncC4.1, RotEncC?.1, RotEncC?.1, SW3.2, SW4.2, TempSensorB1.4 (Pin_4), TempSensorB1.5 (Pin_5), TempSensorC1.4 (Pin_4), TempSensorC1.5 (Pin_5), TempSensorD1.4 (Pin_4), TempSensorD1.5 (Pin_5), U?.4 (GND), USBR1.2
- net SCLSub0: now also LuxSensorA1.2 (Pin_2), TempSensorA1.2 (Pin_2)
- net SCLSub1: now also LuxSensorB1.2 (Pin_2), TempSensorB1.2 (Pin_2)
- net SCLSub2: now also LuxSensorC1.2 (Pin_2), TempSensorC1.2 (Pin_2)
- net SCLSub3: now also LuxSensorD1.2 (Pin_2), R?.2, TempSensorD1.2 (Pin_2)
- net SDASub0: now also LuxSensorA1.1 (Pin_1), TempSensorA1.1 (Pin_1)
- net SDLSub1: now also LuxSensorB1.1 (Pin_1), TempSensorB1.1 (Pin_1)
- net SDLSub2: now also LuxSensorC1.1 (Pin_1), R?.2, R?.2, TempSensorC1.1 (Pin_1)
- net SDLSub3: now also LuxSensorD1.1 (Pin_1), R?.2, TempSensorD1.1 (Pin_1)
- net OUTAIn: now reaches IC1.11 (PD5/T1/OC0B/PCINT21)
- net OUTAIn: now also U?.2 (3Y)
- net OUTBIn: now reaches IC1.12 (PD6/AIN0/OC0A/PCINT22)
- net OUTBIn: now also U?.4 (GND)
- net RotEncSWIn: now reaches IC1.13 (PD7/AIN1/PCINT23)
- net RotEncSWIn: now also U?.7 (1Y)
- net HeatingPadPWM: now reaches IC1.15 (PCINT1/OC1A/PB1)
- net HeatingPadPWM: now also HeaterR1.2
- net HallSensor: now reaches IC1.23 (PCINT8/ADC0/PC0)
- net HallSensor: now also J?.1 (Pin_1)
- net USBCurrentLine1: now reaches IC1.4 (PD2/INT0/PCINT18)
- net USBCurrentLine1: now also EnumR?.1, IC9.9 (PD3(TXD1/INT3))
- net USBCurrentLine2: now reaches IC1.5 (PD3/INT1/OC2B/PCINT19)
- net USBCurrentLine2: now also EnumR?.1, IC9.10 (PD4(INT5/AIN3))
- net LEDOut: now reaches IC1.6 (PD4/T0/XCK/PCINT20)
- net MISO renamed MISO1
- net MISO1: now also PogoPinISR1.2 (Pin_2)
- net MOSI renamed MOSI1
- net MOSI1: now also PogoPinISR1.1 (Pin_1)
- net RESET renamed RESET1
- net RESET1: now also PogoPinISR1.4 (Pin_4), R?.2, SW4.1
- net SCK renamed SCK1
- net SCK1: now also PogoPinISR1.3 (Pin_3)
- new net: IC3.1 (D1), IC3.2 (D1), IC3.3 (S2)
- new net: HeaterR1.1, HeaterR2.1, IC3.4 (G2)
- new net: HE1.2, IC3.7 (S1)
- new net: HeaterR3.2, HeaterR4.2, IC3.8 (G1)
- new net: HE1.1, IC4.1 (OUT), Limiter2C2.1
- new net: FB1.1, Ferrite1C2.1, IC6.1 (OUT)
- new net: IC6.2 (ILIM), R?.1
- new net: IC6.3 (FLAG), IC7.1 (G), Limiter1R3.1
- new net: IC6.4 (EN), Limiter1R1.2
- new net: IC4.2 (ILIM), R?.1
- new net: IC4.3 (FLAG), IC5.1 (G), Limiter1R?.1
- new net: IC4.4 (EN), Limiter2R1.2
- new net: D?.2 (A), IC7.3 (D)
- new net: D?.1 (K), Limiter1R4.1
- new net: D?.2 (A), IC5.3 (D)
- new net: D?.1 (K), Limiter2R4.1
- new net: IC8.5 (Vp(Vcc)), J?.1 (VBUS), SW1.2 (B)
- new net: J?.5 (Shield), USBR1.1
- new net: EnumC3.1, IC9.27 (UCAP)
- new net: EnumR3.1, IC9.29 (D+)
- new net: EnumR2.2, IC9.30 (D-)
- new net: 3.5VBuckC1.1, 3.5VBuckL1.2, IC10.2 (SW)
- new net: 3.5VBuckR1.1, 3.5VBuckR2.1, IC10.4 (VFB)
- new net: 3.5VBuckR1.2, IC10.5 (EN)
- new net: 3.5VBuckC1.2, IC10.6 (VBST)
- new net: IC12.4 (SCLK), TempSensorA2.1 (Pin_1)
- new net: IC12.5 (SDA), TempSensorA2.2 (Pin_2)
- new net: IC12.3 (Vdd), TempAC1.1, TempSensorA2.3 (Pin_3)
- new net: IC12.2 (GND), TempAC1.2, TempSensorA2.4 (Pin_4), TempSensorA2.5 (Pin_5)
- new net: IC13.4 (SDA), LuxSensorA2.1 (Pin_1)
- new net: IC13.1 (SCL), LuxSensorA2.2 (Pin_2)
- new net: IC13.2 (VDD), LuxAC1.2, LuxSensorA2.3 (Pin_3)
- new net: IC13.3 (GND), LuxAC1.1, LuxSensorA2.4 (Pin_4), LuxSensorA2.5 (Pin_5)
- new net: IC14.4 (SCLK), TempSensorB1.1 (Pin_1)
- new net: IC14.5 (SDA), TempSensorB1.2 (Pin_2)
- new net: IC14.3 (Vdd), TempBC1.1, TempSensorB1.3 (Pin_3)
- new net: IC14.2 (GND), TempBC1.2, TempSensorB1.4 (Pin_4), TempSensorB1.5 (Pin_5)
- new net: IC15.3 (GND), LuxBC1.1, LuxSensorB2.4 (Pin_4), LuxSensorB2.5 (Pin_5)
- new net: IC15.2 (VDD), LuxBC1.2, LuxSensorB2.3 (Pin_3)
- new net: IC15.1 (SCL), LuxSensorB2.2 (Pin_2)
- new net: IC15.4 (SDA), LuxSensorB2.1 (Pin_1)
- new net: IC16.4 (SCLK), TempSensorC2.1 (Pin_1)
- new net: IC16.5 (SDA), TempSensorC2.2 (Pin_2)
- new net: IC16.3 (Vdd), TempCC1.1, TempSensorC2.3 (Pin_3)
- new net: IC16.2 (GND), TempCC1.2, TempSensorC2.4 (Pin_4), TempSensorC2.5 (Pin_5)
- new net: IC17.3 (GND), LuxCC1.1, LuxSensorC2.4 (Pin_4), LuxSensorC2.5 (Pin_5)
- new net: IC17.2 (VDD), LuxCC1.2, LuxSensorC2.3 (Pin_3)
- new net: IC17.1 (SCL), LuxSensorC2.2 (Pin_2)
- new net: IC17.4 (SDA), LuxSensorC2.1 (Pin_1)
- new net: IC18.4 (SCLK), TempSensorD2.1 (Pin_1)
- new net: IC18.5 (SDA), TempSensorD2.2 (Pin_2)
- new net: IC18.3 (Vdd), TempDC1.1, TempSensorD2.3 (Pin_3)
- new net: IC18.2 (GND), TempDC1.2, TempSensorD2.4 (Pin_4), TempSensorD2.5 (Pin_5)
- new net: IC19.3 (GND), LuxDC1.1, LuxSensorD2.4 (Pin_4), LuxSensorD2.5 (Pin_5)
- new net: IC19.2 (VDD), LuxDC1.2, LuxSensorD2.3 (Pin_3)
- new net: IC19.1 (SCL), LuxSensorD2.2 (Pin_2)
- new net: IC19.4 (SDA), LuxSensorD2.1 (Pin_1)
- new net: J?.1 (Pin_1), RotEncR?.2, SW5.A
- new net: J?.2 (Pin_2), RotEncR?.2, SW5.B
- new net: J?.5 (Pin_5), J?.6 (Pin_6), SW5.C, SW5.S1
- new net: J?.3 (Pin_3), RotEncR?.2, SW5.S2
- new net: J?.4 (Pin_4), RotEncR?.1, RotEncR?.1, RotEncR?.1
- new net: RotEncC?.2, RotEncR?.2, U?.1 (1A)
- new net: RotEncC?.2, RotEncR?.2, U?.3 (2A)
- new net: RotEncC4.2, RotEncR5.2, U?.6 (3A)
- new net: J?.1 (Pin_1), RotEncR?.1, RotEncR?.2
- new net: J?.2 (Pin_2), RotEncR?.1, RotEncR?.2
- new net: J?.3 (Pin_3), RotEncR5.1, RotEncR6.2
- new net: J?.1 (Pin_1), U?.2 (Out)
- new net: HallC1.2, J?.2 (Pin_2), U?.1 (Vcc)
- new net: HallC1.1, J?.3 (Pin_3), J?.4 (Pin_4), U?.3 (GND)
- new net: PogoPinISR2.1 (Pin_1), U?.2 (A1)
- new net: PogoPinISR2.2 (Pin_2), U?.3 (A2)
- new net: PogoPinISR2.3 (Pin_3), U?.4 (A3)
- new net: PogoPinISR2.4 (Pin_4), U?.5 (A4)
- new net: J?.2 (Pin_2), PogoPinISR2.5 (Pin_5), U?.14 (VccB)
- new net: J?.1 (Pin_1), PogoPinISR2.6 (Pin_6), ProgrammerC2.1, ProgrammerC2.2, ProgrammerC2.2, ProgrammerR1.2, U?.7 (GND)
- new net: PogoPinISR2.7 (Pin_7), ProgrammerC2.1, SW?.2 (B), U?.1 (VccA)
- new net: J?.6 (Pin_6), U?.10 (B4)
- new net: J?.5 (Pin_5), U?.11 (B3)
- new net: J?.4 (Pin_4), U?.12 (B2)
- new net: J?.3 (Pin_3), U?.13 (B1)
- new net: ProgrammerR1.1, SW?.1 (A), U?.8 (OE)
- new net 3.5V: 3.5VBuckC4.1, 3.5VBuckL1.1, 3.5VBuckR2.2, 3VLDOC1.1, IC11.3 (Input)
- new net 5V: 3.5VBuckC2.1, 3.5VBuckC3.1, 3.5VBuckR1.1, EnumC1.1, EnumC2.1, EnumR1.1, EnumR?.2, EnumR?.2, FB1.2, Ferrite1C1.1, IC10.3 (Vin), IC9.31 (UVCC), IC9.32 (AVCC), IC9.4 (VCC), PogoPinISR3.5 (Pin_5), SW2.2 (B)
- new net 5V_USB_In: IC6.6 (IN), IC7.2 (S), Limiter1C1.1, Limiter1C2.1, Limiter1C3.1, Limiter1R1.1, PogoPinISR1.5 (Pin_5), SW1.1 (A)
- new net HeatingPadOnOff: HeaterR3.1
- new net MISO2: IC9.17 ((PCINT3/MISO/PDO)PB3), PogoPinISR3.2 (Pin_2)
- new net MOSI2: IC9.16 (PB2(PDI/MOSI/PCINT2)), PogoPinISR3.1 (Pin_1)
- new net OverCurrentLED2: IC4.6 (IN), IC5.2 (S), Limiter2C1.1, Limiter2R1.1, SW2.1 (A)
- new net RESET2: EnumR1.2, IC9.24 ((PC1/dW)RESET), PogoPinISR3.4 (Pin_4), SW3.1
- new net SCK2: IC9.15 (PB1(SCLK/PCINT1)), PogoPinISR3.3 (Pin_3)
- new net USBD+: EnumR3.2, IC8.6 (I/O4), J?.3 (D+)
- new net USBD-: EnumR2.1, IC8.4 (I/O3), J?.2 (D-)
- new net XTAL1: EnumC5.1, EnumCrystal1.1, IC9.1 (XTAL1)
- new net XTAL2: EnumC4.1, EnumCrystal1.3, IC9.2 (XTAL2(PC0))
Other:
- note added: "28F0181-1SR-10"
- note added: "Current and Inrush Limiting and Filtering"
- note added: "Enumeration IC"
- note added: "Heating Control and Power Regulation"
- note added: "Heating Pad Control and Redundant Current Limiting"
- note added: "If too much input capacitance draws too much\ncurrent and crashes the USB port, replace \nwith smaller capacitors. Shouldn't be a problem \nsince the NCP380 current limiter has soft\nstart."
- note added: "Main Controller"
- note added: "Note: 5th pins are for cable shielding"
- note added: "Note: Debounce circuit not finalized, may be changed."
- note added: "Note: These values were auto-generated \nby TI WEBENCH Power Designer and need \nto be verifed before these values are finalized."
- note added: "Note: pushbutton still needs to be tested."
- note added: "Optional resistor to dampen EM emissions"
- note added: "Peripherals and Daughter Boards"
- note added: "Resistance vale to be decided."
- note added: "These resistance values need to be tested\nwith this mosfet"
- note added: "This resistance depends on the power pack supply. \nUse a 44kOhm resistor for 0.5A, or a higher one.\nValue to be decided."
- note added: "To 5V ISR programmer"
- note added: "Turn on LED on overcurrent fault"
- note added: "USB Input"
- note added: "Use two pulled up IO lines to signal main IC amount of \ncurrent is avaliable."
- note added: "Used for USB enumeration to get 500mA or higher\n"
- note added: "Used for programming enumeration chip."
- note added: "Used for programming the board. The signal pins are all 3V, the power is 5V."
- note added: "Using this chip for ease of soldering.\nTo use full speed USB use a TSV diode meant for USB."
- note added: "Voltage Regulation"
- note removed: "Used for programming the board."
- moved on the sheet: BluC1, I2CHubC1, I2CHubR1, I2CHubR2, IC1, IC2, JY-MCUBluetooth, LuxSensorA1, OLEDC1, OLEDModule, R?, SCLR1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
